File: mirakeeb.kicad_sch (KiCad schematic)
At the start: 76 parts, among them J1 OLED_128x64, SW1 RotaryEncoder_Switch, SW2 RotaryEncoder_Switch, U1 Raspberry_Pi_Pico

Commit message: more stuff
Parts:
- removed SW2: RotaryEncoder_Switch, symbol Device:RotaryEncoder_Switch
- added D38, D39, D40, D41, D42, D43, D44, D45, D46, D47, D48, D49: Diode, ScottoKeebs_Components:Diode_DO-35, symbol ScottoKeebs:Placeholder_Diode
- added D50, D51, D52, D53, D54, D55, D56, D57, D58, D59, D60, D61, D62, D63, D64, D65, D66, D67, D68, D69, D70, D71, D72, D73, D74, D75, D76, D77, D78, D79, D80, D81, D82, D83, D84, D85, D86, D87, D88, D89, D90, D91, D92, D93, D94, D95, D96, D97: LED_SK6812MINI, ScottoKeebs_Components:LED_SK6812MINI, symbol ScottoKeebs:LED_SK6812MINI
- added S37, S38, S39, S40, S41, S42, S43, S44, S45, S46, S47, S48: Keyswitch, symbol ScottoKeebs:Placeholder_Keyswitch
- added SW2: RotaryEncoder, Rotary_Encoder:RotaryEncoder_Bourns_Horizontal_PEC09-2xxxF-Nxxxx, symbol Device:RotaryEncoder
Connections:
- net C0: now also U1.14 (GPIO10), S45.1, S46.1, S47.1, S48.1; no longer S1.1, S11.1, S6.1
- net C1: now also S17.1, S18.1, U1.15 (GPIO11), S43.1, S44.1; no longer S12.1, S2.1, S7.1
- net C2: now also S14.1, S15.1, S16.1, U1.16 (GPIO12); no longer S18.1, S3.1, S8.1
- net C3: now also S10.1, S11.1, S12.1, U1.17 (GPIO13); no longer S14.1, S16.1, S4.1
- net C4: now also S6.1, S7.1, S8.1, U1.19 (GPIO14); no longer S10.1, S15.1, S17.1
- net C5: now also S1.1, S2.1, S3.1, S4.1, U1.20 (GPIO15); no longer S33.1, S34.1, S35.1, S36.1
- net C6: now also S33.1, S34.1, S35.1, S36.1, U1.21 (GPIO16); no longer S29.1, S30.1, S31.1, S32.1
- net C7: now also S29.1, S30.1, S31.1, S32.1, U1.22 (GPIO17); no longer S25.1, S26.1, S27.1, S28.1
- net C8: now also S25.1, S26.1, S27.1, S28.1, U1.24 (GPIO18); no longer S22.1, S23.1, S24.1
- net C9: now also S22.1, S23.1, S24.1, U1.25 (GPIO19), S40.1; no longer S19.1, S20.1, S21.1
- net R0: now also D13.1 (K), D17.1 (K), D9.1 (K), U1.9 (GPIO6), D38.1 (K), D46.1 (K); no longer D2.1 (K), D3.1 (K), D4.1 (K)
- net R1: now also D14.1 (K), D18.1 (K), D2.1 (K), U1.10 (GPIO7), D39.1 (K), D47.1 (K); no longer D7.1 (K), D8.1 (K), D9.1 (K)
- net R2: now also D3.1 (K), D7.1 (K), U1.11 (GPIO8), D40.1 (K), D44.1 (K), D48.1 (K); no longer D12.1 (K), D13.1 (K), D14.1 (K)
- net R3: now also D12.1 (K), D4.1 (K), D8.1 (K), U1.12 (GPIO9), D41.1 (K), D42.1 (K), D43.1 (K), D45.1 (K), D49.1 (K); no longer D17.1 (K), D18.1 (K)
- net GND: now reaches U1.13 (GND)
- net GND: now also SW1.C, U1.18 (GND), U1.23 (GND), U1.28 (GND), U1.3 (GND), U1.38 (GND), U1.8 (GND), SW2.C
- net c10: now reaches U1.26 (GPIO20)
- net c10: now also S19.1, S20.1, S21.1, S41.1
- net c11: now reaches U1.27 (GPIO21)
- net c11: now also S37.1, S38.1, S39.1, S42.1
- new net: D88.1 (DOUT), D92.3 (DIN)
- new net: D88.2 (VSS), D89.4 (VDD)
- new net: D84.1 (DOUT), D88.3 (DIN)
- new net: D87.2 (VSS), D88.4 (VDD)
- new net: D48.2 (A), S47.2
- new net: D55.1 (DOUT), D62.3 (DIN)
- new net: D55.2 (VSS), D62.4 (VDD)
- new net: D54.1 (DOUT), D55.3 (DIN)
- new net: D70.1 (DOUT), D72.3 (DIN)
- new net: D70.2 (VSS), D77.4 (VDD)
- new net: D68.1 (DOUT), D70.3 (DIN)
- new net: D66.2 (VSS), D70.4 (VDD)
- new net: D49.2 (A), S48.2
- new net: D75.1 (DOUT), D77.3 (DIN)
- new net: D73.1 (DOUT), D75.3 (DIN)
- new net: D72.2 (VSS), D75.4 (VDD)
- new net: D71.1 (DOUT), D73.3 (DIN)
- new net: D69.1 (DOUT), D71.3 (DIN)
- new net: D71.4 (VDD), D76.2 (VSS)
- new net: D86.1 (DOUT), D90.3 (DIN)
- new net: D86.2 (VSS), D87.4 (VDD)
- new net: D82.1 (DOUT), D86.3 (DIN)
- new net: D94.1 (DOUT), D95.3 (DIN)
- new net: D94.2 (VSS), D95.4 (VDD)
- new net: D90.1 (DOUT), D94.3 (DIN)
- new net: D83.3 (DIN), D87.1 (DOUT)
- new net: D87.3 (DIN), D91.1 (DOUT)
- new net: D65.1 (DOUT), D66.3 (DIN)
- new net: D65.2 (VSS), D72.4 (VDD)
- new net: D64.1 (DOUT), D65.3 (DIN)
- new net: D52.2 (VSS), D65.4 (VDD)
- new net: D47.2 (A), S46.2
- new net: D39.2 (A), S38.2
- new net: D53.1 (DOUT), D54.3 (DIN)
- new net: D53.2 (VSS), D64.4 (VDD)
- new net: D52.1 (DOUT), D53.3 (DIN)
- new net: D62.1 (DOUT), D63.3 (DIN)
- new net: D62.2 (VSS), D78.4 (VDD)
- new net: D80.1 (DOUT), D84.3 (DIN)
- new net: D80.2 (VSS), D81.4 (VDD)
- new net: D58.1 (DOUT), D80.3 (DIN)
- new net: D61.2 (VSS), D80.4 (VDD)
- new net: D73.4 (VDD), D74.2 (VSS)
- new net: D38.2 (A), S37.2
- new net: D40.2 (A), S39.2
- new net: D44.2 (A), S43.2
- new net: D57.1 (DOUT), D58.3 (DIN)
- new net: D57.2 (VSS), D58.4 (VDD)
- new net: D57.3 (DIN), D61.1 (DOUT)
- new net: D56.2 (VSS), D57.4 (VDD)
- new net: D84.2 (VSS), D85.4 (VDD)
- new net: D83.2 (VSS), D84.4 (VDD)
- new net: D61.3 (DIN), D83.1 (DOUT)
- new net: D60.2 (VSS), D61.4 (VDD)
- new net: D69.3 (DIN), D78.1 (DOUT)
- new net: D69.4 (VDD), D78.2 (VSS)
- new net: D76.1 (DOUT), D78.3 (DIN)
- new net: D77.1 (DOUT), D79.3 (DIN)
- new net: D68.2 (VSS), D79.4 (VDD)
- new net: D82.2 (VSS), D83.4 (VDD)
- new net: D74.1 (DOUT), D76.3 (DIN)
- new net: D72.1 (DOUT), D74.3 (DIN)
- new net: D64.2 (VSS), D74.4 (VDD)
- new net: D43.2 (A), S42.2
- new net: D51.1 (DOUT), D52.3 (DIN)
- new net: D51.2 (VSS), D66.4 (VDD)
- new net: D50.1 (DOUT), D51.3 (DIN)
- new net: D50.2 (VSS), D67.4 (VDD)
- new net: D59.3 (DIN), D81.1 (DOUT)
- new net: D81.3 (DIN), D85.1 (DOUT)
- new net: D93.3 (DIN), D97.1 (DOUT)
- new net: D96.1 (DOUT), D97.3 (DIN)
- new net: D96.2 (VSS), D97.4 (VDD)
- new net: D91.2 (VSS), D92.4 (VDD)
- new net: D91.3 (DIN), D95.1 (DOUT)
- new net: D90.2 (VSS), D91.4 (VDD)
- new net: D45.2 (A), S44.2
- new net: D66.1 (DOUT), D67.3 (DIN)
- new net: D85.3 (DIN), D89.1 (DOUT)
- new net: D67.1 (DOUT), D68.3 (DIN)
- new net: D67.2 (VSS), D68.4 (VDD)
- new net: D92.1 (DOUT), D96.3 (DIN)
- new net: D92.2 (VSS), D93.4 (VDD)
- new net: D56.1 (DOUT), D60.3 (DIN)
- new net: D41.2 (A), S40.2
- new net: D89.3 (DIN), D93.1 (DOUT)
- new net: D63.1 (DOUT), D64.3 (DIN)
- new net: D63.2 (VSS), D76.4 (VDD)
- new net: D54.2 (VSS), D63.4 (VDD)
- new net: D95.2 (VSS), D96.4 (VDD)
- new net: D58.2 (VSS), D59.4 (VDD)
- new net: D46.2 (A), S45.2
- new net: D42.2 (A), S41.2
- new net: D60.1 (DOUT), D82.3 (DIN)
Other:
- moved on the sheet: SW1

Commit message: asdf
Connections:
- net GND: now also D59.2 (VSS), D69.2 (VSS), D71.2 (VSS), D73.2 (VSS), D75.2 (VSS), D77.2 (VSS), D79.2 (VSS), D81.2 (VSS), D85.2 (VSS), D89.2 (VSS), D93.2 (VSS), D97.2 (VSS)
- net at U1.1 (GPIO0): now also SW2.B
- net at U1.2 (GPIO1): now also SW2.A
- net at U1.4 (GPIO2): now also SW1.B
- net at U1.5 (GPIO3): now also SW1.A
- net sda: now reaches U1.6 (GPIO4)
- net sda: now also J1.4 (SDA)
- net scl: now reaches U1.7 (GPIO5)
- net scl: now also J1.3 (SCL)

Commit message: ping
Parts:
- S1, S10, S11, S12, S13, S14, S15, S16, S17, S18, S19, S2, S20, S21, S22, S23, S24, S25, S26, S27, S28, S29, S3, S30, S31, S32, S33, S34, S35, S36, S37, S38, S39, S4, S40, S41, S42, S43, S44, S45, S46, S47, S48, S5, S6, S7, S8, S9: footprint (none) -> ScottoKeebs_MX:MX_PCB
- SW1: footprint (none) -> Rotary_Encoder:RotaryEncoder_Alps_EC11E-Switch_Vertical_H20mm
Connections:
- net GND: now also J1.1 (GND)
- net ledhalf0: now reaches U1.29 (GPIO22)
- net ledhalf0: now also D50.3 (DIN)
- net at U1.34 (GPIO28_ADC2): now also SW1.S2
- net +3.3V: now reaches U1.36 (3V3)
- net +3.3V: now also SW1.S1
- net +5V: now reaches U1.40 (VBUS)
- net +5V: now also D50.4 (VDD), D51.4 (VDD), D52.4 (VDD), D53.4 (VDD), D54.4 (VDD), D55.4 (VDD), D56.4 (VDD), D60.4 (VDD), D82.4 (VDD), D86.4 (VDD), D90.4 (VDD), D94.4 (VDD), J1.2 (VCC)
- net at D79.1 (DOUT): now also D56.3 (DIN)
- no-connect marks 0 -> 12
Other:
- moved on the sheet: D50, D51, D52, D53, D54, D55, D62, D63, D64, D65, D66, D67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

Commit message: pretty much final design, just need graphics
Parts:
- D1, D10, D11, D12, D13, D14, D15, D16, D17, D18, D19, D2, D20, D21, D22, D23, D24, D25, D26, D27, D28, D29, D3, D30, D31, D32, D33, D34, D35, D36, D38, D39, D4, D40, D41, D42, D43, D44, D45, D46, D47, D48, D49, D5, D6, D7, D8, D9: footprint ScottoKeebs_Components:Diode_DO-35 -> scotto_components:Diode_DO-35
- D50, D51, D52, D53, D54, D55, D56, D57, D58, D59, D60, D61, D62, D63, D64, D65, D66, D67, D68, D69, D70, D71, D72, D73, D74, D75, D76, D77, D78, D79, D80, D81, D82, D83, D84, D85, D86, D87, D88, D89, D90, D91, D92, D93, D94, D95, D96, D97: footprint ScottoKeebs_Components:LED_SK6812MINI -> scotto_components:LED_SK6812MINI
- J1: footprint ScottoKeebs_Components:OLED_128x64 -> scotto_components:OLED_128x64
- S1, S10, S11, S12, S13, S14, S15, S16, S17, S18, S19, S2, S20, S21, S22, S23, S24, S25, S26, S27, S28, S29, S3, S30, S31, S32, S33, S34, S35, S36, S37, S38, S39, S4, S40, S41, S42, S43, S44, S45, S46, S47, S48, S5, S6, S7, S8, S9: footprint ScottoKeebs_MX:MX_PCB -> mx_keebs:MX_PCB_1.00u
Connections:
- net +5V: now also D57.4 (VDD), D58.4 (VDD), D59.4 (VDD), D61.4 (VDD), D62.4 (VDD), D63.4 (VDD), D64.4 (VDD), D65.4 (VDD), D66.4 (VDD), D67.4 (VDD), D68.4 (VDD), D69.4 (VDD), D70.4 (VDD), D71.4 (VDD), D72.4 (VDD), D73.4 (VDD), D74.4 (VDD), D75.4 (VDD), D76.4 (VDD), D77.4 (VDD), D78.4 (VDD), D79.4 (VDD), D80.4 (VDD), D81.4 (VDD), D83.4 (VDD), D84.4 (VDD), D85.4 (VDD), D87.4 (VDD), D88.4 (VDD), D89.4 (VDD), D91.4 (VDD), D92.4 (VDD), D93.4 (VDD), D95.4 (VDD), D96.4 (VDD), D97.4 (VDD)
- net GND: now also D50.2 (VSS), D51.2 (VSS), D52.2 (VSS), D53.2 (VSS), D54.2 (VSS), D55.2 (VSS), D56.2 (VSS), D57.2 (VSS), D58.2 (VSS), D60.2 (VSS), D61.2 (VSS), D62.2 (VSS), D63.2 (VSS), D64.2 (VSS), D65.2 (VSS), D66.2 (VSS), D67.2 (VSS), D68.2 (VSS), D70.2 (VSS), D72.2 (VSS), D74.2 (VSS), D76.2 (VSS), D78.2 (VSS), D80.2 (VSS), D82.2 (VSS), D83.2 (VSS), D84.2 (VSS), D86.2 (VSS), D87.2 (VSS), D88.2 (VSS), D90.2 (VSS), D91.2 (VSS), D92.2 (VSS), D94.2 (VSS), D95.2 (VSS), D96.2 (VSS)
- no-connect marks 12 -> 11
Other:
- moved on the sheet: D50, D51, D52, D53, D54, D55, D56, D57, D58, D59, D60, D61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
