File: mirakeeb.kicad_pcb (KiCad board)
At the start: 2 copper layers, 3.4 x 3 mm, 148 parts, among them J1 OLED_128x64, SW1 RotaryEncoder_Switch, SW2 RotaryEncoder, U1 Raspberry_Pi_Pico

Commit message: pong
Parts:
- moved S4 43.7 mm to (133.3, 58.4)
- moved S10 43.2 mm to (61.8, 81.0)
- moved S5 43.2 mm to (76.3, 66.4)
- moved S7 43.2 mm to (76.3, 95.5)
- moved S8 43.2 mm to (76.3, 110.0)
- moved S11 43.2 mm to (61.8, 95.5)
- moved S12 43.2 mm to (61.8, 110.0)
- moved S9 43.2 mm to (61.8, 66.4)
- moved S6 43.1 mm to (76.3, 81.0)
- moved S3 2.09 mm to (133.3, 89.6)
- moved S2 0.23 mm to (133.3, 73.2)
Changed lines of the file:
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@@
 		(pad_to_mask_clearance 0)
 		(allow_soldermask_bridges_in_footprints no)
+		(grid_origin 126.04 51.19)
 		(pcbplotparams
 			(layerselection 0x00010fc_ffffffff)
@@
 	(footprint "ScottoKeebs_MX:MX_PCB"
 		(layer "F.Cu")
-		(at 133.29 102.12)
+		(at 133.29 58.44)
 		(descr "MX keyswitch PCB Mount")
 		(tags "MX Keyboard Keyswitch Switch PCB Cutout")
@@
 	(footprint "ScottoKeebs_MX:MX_PCB"
 		(layer "F.Cu")
-		(at 104.2 102.13)
+		(at 61.78 110.04)
 		(descr "MX keyswitch PCB Mount")
 		(tags "MX Keyboard Keyswitch Switch PCB Cutout")
@@
 	(footprint "ScottoKeebs_MX:MX_PCB"
 		(layer "F.Cu")
-		(at 133.29 87.55)
+		(at 133.29 89.64)
 		(descr "MX keyswitch PCB Mount")
 		(tags "MX Keyboard Keyswitch Switch PCB Cutout")
@@
 	(footprint "ScottoKeebs_MX:MX_PCB"
 		(layer "F.Cu")
-		(at 118.73 102.11)
+		(at 76.31 110.04)
 		(descr "MX keyswitch PCB Mount")
 		(tags "MX Keyboard Keyswitch Switch PCB Cutout")
@@
 	(footprint "ScottoKeebs_MX:MX_PCB"
 		(layer "F.Cu")
-		(at 118.73 73)
+		(at 76.325 80.95)
 		(descr "MX keyswitch PCB Mount")
 		(tags "MX Keyboard Keyswitch Switch PCB Cutout")
@@
 	(footprint "ScottoKeebs_MX:MX_PCB"
 		(layer "F.Cu")
-		(at 133.29 73)
+		(at 133.29 73.23)
 		(descr "MX keyswitch PCB Mount")
 		(tags "MX Keyboard Keyswitch Switch PCB Cutout")
@@
 	(footprint "ScottoKeebs_MX:MX_PCB"
 		(layer "F.Cu")
-		(at 118.73 87.55)
+		(at 76.31 95.48)
 		(descr "MX keyswitch PCB Mount")
 		(tags "MX Keyboard Keyswitch Switch PCB Cutout")
@@
 	(footprint "ScottoKeebs_MX:MX_PCB"
 		(layer "F.Cu")
-		(at 104.2 73.02)
+		(at 61.78 80.95)
 		(descr "MX keyswitch PCB Mount")
 		(tags "MX Keyboard Keyswitch Switch PCB Cutout")
@@
 	(footprint "ScottoKeebs_MX:MX_PCB"
 		(layer "F.Cu")
-		(at 118.73 58.44)
+		(at 76.31 66.37)
 		(descr "MX keyswitch PCB Mount")
 		(tags "MX Keyboard Keyswitch Switch PCB Cutout")
@@
 	(footprint "ScottoKeebs_MX:MX_PCB"
 		(layer "F.Cu")
-		(at 104.2 87.57)
+		(at 61.78 95.48)
 		(descr "MX keyswitch PCB Mount")
 		(tags "MX Keyboard Keyswitch Switch PCB Cutout")
@@
 	(footprint "ScottoKeebs_MX:MX_PCB"
 		(layer "F.Cu")
-		(at 104.2 58.46)
+		(at 61.78 66.37)
 		(descr "MX keyswitch PCB Mount")
 		(tags "MX Keyboard Keyswitch Switch PCB Cutout")

Commit message: pretty much final design, just need graphics
Parts:
- D1, D10, D11, D12, D13, D14, D15, D16, D17, D18, D19, D2, D20, D21, D22, D23, D24, D25, D26, D27, D28, D29, D3, D30, D31, D32, D33, D34, D35, D36, D38, D39, D4, D40, D41, D42, D43, D44, D45, D46, D47, D48, D49, D5, D6, D7, D8, D9: footprint ScottoKeebs_Components:Diode_DO-35 -> scotto_components:Diode_DO-35
- D50, D51, D52, D53, D54, D55, D56, D57, D58, D59, D60, D61, D62, D63, D64, D65, D66, D67, D68, D69, D70, D71, D72, D73, D74, D75, D76, D77, D78, D79, D80, D81, D82, D83, D84, D85, D86, D87, D88, D89, D90, D91, D92, D93, D94, D95, D96, D97: footprint ScottoKeebs_Components:LED_SK6812MINI -> scotto_components:LED_SK6812MINI
- J1: footprint ScottoKeebs_Components:OLED_128x64 -> scotto_components:OLED_128x64
- S1, S10, S11, S12, S13, S14, S15, S16, S17, S18, S19, S2, S20, S21, S22, S23, S24, S25, S26, S27, S28, S29, S3, S30, S31, S32, S33, S34, S35, S36, S37, S38, S39, S4, S40, S41, S42, S43, S44, S45, S46, S47, S48, S5, S6, S7, S8, S9: footprint ScottoKeebs_MX:MX_PCB -> mx_keebs:MX_PCB_1.00u
- moved D94 380.0 mm to (300.0, 59.2)
- moved D95 378.1 mm to (300.0, 78.3), turned to 180 degrees
- moved D96 376.7 mm to (300.0, 97.3)
- moved D97 375.9 mm to (300.0, 116.4), turned to 180 degrees
- moved D90 358.3 mm to (280.9, 63.2)
- moved D91 357.2 mm to (280.9, 82.3), turned to 180 degrees
- moved D93 356.7 mm to (280.9, 120.4), turned to 180 degrees
- moved D92 356.6 mm to (280.9, 101.3)
- moved D86 351.0 mm to (261.9, 63.2)
- moved D87 348.7 mm to (261.9, 82.3), turned to 180 degrees
- moved D88 347.0 mm to (261.9, 101.3)
- moved D89 345.9 mm to (261.9, 120.4), turned to 180 degrees
- moved D19 335.5 mm to (271.4, 63.2), turned to 90 degrees
- moved D20 333.2 mm to (271.4, 82.3), turned to 90 degrees
- moved D21 331.7 mm to (271.4, 101.3), turned to 90 degrees
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Connections:
- D50 pad 2: Net-(D50-VSS) -> GND
- D51 pad 2: Net-(D51-VSS) -> GND
- D52 pad 2: Net-(D52-VSS) -> GND
- D53 pad 2: Net-(D53-VSS) -> GND
- D54 pad 2: Net-(D54-VSS) -> GND
- D55 pad 2: Net-(D55-VSS) -> GND
- D56 pad 2: Net-(D56-VSS) -> GND
- D57 pad 2: Net-(D57-VSS) -> GND
- D57 pad 4: Net-(D56-VSS) -> +5V
- D58 pad 2: Net-(D58-VSS) -> GND
- D58 pad 4: Net-(D57-VSS) -> +5V
- D59 pad 4: Net-(D58-VSS) -> +5V
- D60 pad 2: Net-(D60-VSS) -> GND
- D61 pad 2: Net-(D61-VSS) -> GND
- D61 pad 4: Net-(D60-VSS) -> +5V
- D62 pad 2: Net-(D62-VSS) -> GND
- D62 pad 4: Net-(D55-VSS) -> +5V
- D63 pad 2: Net-(D63-VSS) -> GND
- D63 pad 4: Net-(D54-VSS) -> +5V
- D64 pad 2: Net-(D64-VSS) -> GND
- D64 pad 4: Net-(D53-VSS) -> +5V
- D65 pad 2: Net-(D65-VSS) -> GND
- D65 pad 4: Net-(D52-VSS) -> +5V
- D66 pad 2: Net-(D66-VSS) -> GND
- D66 pad 4: Net-(D51-VSS) -> +5V
- D67 pad 2: Net-(D67-VSS) -> GND
- D67 pad 4: Net-(D50-VSS) -> +5V
- D68 pad 2: Net-(D68-VSS) -> GND
- D68 pad 4: Net-(D67-VSS) -> +5V
- D69 pad 4: Net-(D69-VDD) -> +5V
- D70 pad 2: Net-(D70-VSS) -> GND
- D70 pad 4: Net-(D66-VSS) -> +5V
- D71 pad 4: Net-(D71-VDD) -> +5V
- D72 pad 2: Net-(D72-VSS) -> GND
- D72 pad 4: Net-(D65-VSS) -> +5V
- D73 pad 4: Net-(D73-VDD) -> +5V
- D74 pad 2: Net-(D73-VDD) -> GND
- D74 pad 4: Net-(D64-VSS) -> +5V
- D75 pad 4: Net-(D72-VSS) -> +5V
- D76 pad 2: Net-(D71-VDD) -> GND
- D76 pad 4: Net-(D63-VSS) -> +5V
- D77 pad 4: Net-(D70-VSS) -> +5V
- D78 pad 2: Net-(D69-VDD) -> GND
- D78 pad 4: Net-(D62-VSS) -> +5V
- D79 pad 4: Net-(D68-VSS) -> +5V
- D80 pad 2: Net-(D80-VSS) -> GND
- D80 pad 4: Net-(D61-VSS) -> +5V
- D81 pad 4: Net-(D80-VSS) -> +5V
- D82 pad 2: Net-(D82-VSS) -> GND
- D83 pad 2: Net-(D83-VSS) -> GND
- D83 pad 4: Net-(D82-VSS) -> +5V
- D84 pad 2: Net-(D84-VSS) -> GND
- D84 pad 4: Net-(D83-VSS) -> +5V
- D85 pad 4: Net-(D84-VSS) -> +5V
- D86 pad 2: Net-(D86-VSS) -> GND
- D87 pad 2: Net-(D87-VSS) -> GND
- D87 pad 4: Net-(D86-VSS) -> +5V
- D88 pad 2: Net-(D88-VSS) -> GND
- D88 pad 4: Net-(D87-VSS) -> +5V
- D89 pad 4: Net-(D88-VSS) -> +5V
- D90 pad 2: Net-(D90-VSS) -> GND
- D91 pad 2: Net-(D91-VSS) -> GND
- D91 pad 4: Net-(D90-VSS) -> +5V
- D92 pad 2: Net-(D92-VSS) -> GND
- D92 pad 4: Net-(D91-VSS) -> +5V
- D93 pad 4: Net-(D92-VSS) -> +5V
- D94 pad 2: Net-(D94-VSS) -> GND
- D95 pad 2: Net-(D95-VSS) -> GND
- D95 pad 4: Net-(D94-VSS) -> +5V
- D96 pad 2: Net-(D96-VSS) -> GND
- D96 pad 4: Net-(D95-VSS) -> +5V
- D97 pad 4: Net-(D96-VSS) -> +5V
Routing:
- net R3: track 0.00 -> 364.7 mm, vias 0 -> 1
- net R2: track 0.00 -> 320.3 mm, vias 0 -> 1
- net R1: track 0.00 -> 304.4 mm, vias 0 -> 2
- net R0: track 0.00 -> 276.1 mm, vias 0 -> 2
- net C1: track 0.00 -> 208.8 mm
- net C0: track 0.00 -> 193.2 mm
- net c11: track 0.00 -> 178.2 mm
- net Net-(U1-GPIO0): track 0.00 -> 156.1 mm, vias 0 -> 2
- net c10: track 0.00 -> 155.0 mm, vias 0 -> 2
- net Net-(U1-GPIO1): track 0.00 -> 154.3 mm, vias 0 -> 2
- net C2: track 0.00 -> 150.3 mm
- net C9: track 0.00 -> 138.6 mm, vias 0 -> 1
- net C5: track 0.00 -> 130.7 mm, vias 0 -> 3
- net C3: track 0.00 -> 130.2 mm
- net C4: track 0.00 -> 127.6 mm, vias 0 -> 1
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- added copper zone on F.Cu, net +5V
- added copper zone on B.Cu, net GND
Other:
- board size 3.4 x 3 mm -> 300 x 140.5 mm
- board text added: "11-14 m/s = Svu (Swallow velocity, unladen)"
- board text added: "It was Walpole"
- board text added: "Made by M1racl3max"
- board text added: "Speak friend and enter"
- board text added: "The Mirakeeb Walpole"

Commit message: graphics
Other:
- board text added: "Ash nazg durbatulûk, ash nazg gimbatul, ash nazg thrakatulûk, agh burzum-ishi krimpatul"

Commit message: ack
Parts:
- moved J1 2.38 mm to (169.0, 115.6)
- moved U1 2.38 mm to (169.0, 53.7)
- turned SW2 to 40 degrees
Routing:
- net scl: track 84.3 -> 74.0 mm, vias 3 -> 2
- net R3: track 364.7 -> 372.2 mm, vias 1 -> 2
- net sda: track 75.4 -> 81.1 mm
- net ledhalf0: track 55.1 -> 58.7 mm, vias 2 -> 1
- net Net-(U1-GPIO0): track 156.1 -> 159.0 mm
- net Net-(U1-GPIO1): track 154.3 -> 157.1 mm
- net R2: track 320.3 -> 317.7 mm
- net c11: track 178.2 -> 180.6 mm
- net Net-(U1-GPIO3): track 27.6 -> 25.2 mm
- net Net-(U1-GPIO28_ADC2): track 48.7 -> 46.4 mm
- net Net-(U1-GPIO2): track 22.6 -> 20.2 mm
- net C3: track 130.2 -> 127.9 mm
- net +3.3V: track 42.7 -> 40.3 mm
- net C4: track 127.6 -> 125.5 mm
- net C2: track 150.3 -> 148.4 mm
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